File: Hardware/PCB/KiCad project/Main_PCB_LF_3.0/Main_PCB_GRUZIK_3.0/Main_PCB_GRUZIK_3.0.kicad_sch (KiCad schematic)
At the start: 63 parts, among them J1 +VIN-, J2 Micro_SD_Card, P1 Conn_01x01, P2 Conn_01x01, P3 Conn_01x01, P4 Conn_01x01, SW1 SW_SPST, SW2 SW_DPDT_x2, U1 STM32G474RETx, U2 AMS1117-5.0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

Commit message: New motors and modes
Other:
- note added: "LiPo 7,4V JST connector"
- note removed: "LiPo 7,4V JST connector with 2x 0,5A diodes"
Changed lines of the file:
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@@
 		)
 	)
-	(text "LiPo 7,4V JST connector\nwith 2x 0,5A diodes"
+	(text "LiPo 7,4V JST connector\n"
 		(exclude_from_sim no)
-		(at 263.906 112.522 0)
+		(at 264.414 108.966 0)
 		(effects
 			(font
@@
 	(label "HSE_IN"
 		(at 97.79 68.834 0)
-		(fields_autoplaced yes)
 		(effects
 			(font
@@
 	(label "LSE_OUT"
 		(at 95.758 119.634 0)
-		(fields_autoplaced yes)
 		(effects
 			(font
@@
 	(label "HSE_OUT"
 		(at 97.79 71.374 0)
-		(fields_autoplaced yes)
 		(effects
 			(font
@@
 	(label "LSE_IN"
 		(at 95.758 117.094 0)
-		(fields_autoplaced yes)
 		(effects
 			(font
